File: content/post/week-8/qtouch-board/qtouch-board.kicad_pcb (KiCad board)
At the start: 2 copper layers, 18 parts, among them J1 Conn_PinSocket_1x05_P2.54mm_V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, J2 Conn_PinSocket_1x02_P2.54mm_V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, J3 Conn_PinSocket_1x03_P2.54mm_V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, J4 Conn_PinSocket_1x02_P2.54mm_V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, SW1 Switch_Slide_Top_CnK, SW2 Switch_Slide_Top_CnK, U1 SeeeduinoXIAO

Commit message: Catching up with documentation for weeks 7 and 8
Parts:
- added H1: MountingHole_M3, fab:MountingHole_M3, F.Cu at (158.0, 55.0)
- added H2: MountingHole_M3, fab:MountingHole_M3, F.Cu at (66.0, 102.0)
- added H3: MountingHole_M3, fab:MountingHole_M3, F.Cu at (197.0, 102.0)
- added J10: Conn_PinHeader_1x01_P2.54mm_Vertical_THT_D1mm, fab:PinHeader_1x01_P2.54mm_Vertical_THT_D1mm, F.Cu at (171.5, 109.0)
- added J11: Conn_PinHeader_1x01_P2.54mm_Vertical_THT_D1mm, fab:PinHeader_1x01_P2.54mm_Vertical_THT_D1mm, F.Cu at (191.5, 109.0)
- added J5: Conn_Header_JST_PH_1x04_P2mm_Vertical_SMD, fab:Header_JST_PH_1x04_P2mm_Vertical_SMD, F.Cu at (89.0, 78.0)
- added J6: Conn_PinHeader_1x01_P2.54mm_Vertical_THT_D1mm, fab:PinHeader_1x01_P2.54mm_Vertical_THT_D1mm, F.Cu at (91.5, 109.0)
- added J7: Conn_PinHeader_1x01_P2.54mm_Vertical_THT_D1mm, fab:PinHeader_1x01_P2.54mm_Vertical_THT_D1mm, F.Cu at (111.5, 109.0)
- added J8: Conn_PinHeader_1x01_P2.54mm_Vertical_THT_D1mm, fab:PinHeader_1x01_P2.54mm_Vertical_THT_D1mm, F.Cu at (131.5, 109.0)
- added J9: Conn_PinHeader_1x01_P2.54mm_Vertical_THT_D1mm, fab:PinHeader_1x01_P2.54mm_Vertical_THT_D1mm, F.Cu at (151.5, 109.0)
- J4: value Conn_PinSocket_1x02_P2.54mm_Vertical_SMD -> Conn_PinHeader_1x01_P2.54mm_Vertical_THT_D1mm; footprint fab:PinSocket_1x02_P2.54mm_Vertical_SMD -> fab:PinHeader_1x01_P2.54mm_Vertical_THT_D1mm
- moved J4 36.9 mm to (71.5, 109.0), turned to 0 degrees
- moved J2 27.0 mm to (124.8, 97.0)
- moved J1 11.4 mm to (133.9, 97.0), turned to 90 degrees
- moved SW2 5.51 mm to (100.0, 75.5)
- moved R4 5.10 mm to (145.0, 63.0)
- moved SW1 4.78 mm to (100.0, 84.5)
- moved R3 3.45 mm to (110.0, 76.0)
- moved J3 2.00 mm to (67.0, 57.0)
- moved R1 1.97 mm to (110.0, 68.0)
- moved R2 1.97 mm to (110.0, 72.0)
- moved D1 1.63 mm to (117.2, 73.8)
- moved D2 1.63 mm to (122.0, 73.8)
- moved D4 1.63 mm to (132.0, 73.7)
- moved D5 1.63 mm to (137.0, 73.7)
- moved D6 1.63 mm to (142.0, 73.7)
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Connections:
- J1 pad 1: QT7_MOSI -> QT3_TX
- J1 pad 2: QT6_MISO -> QT4_RX
- J1 pad 4: QT4_RX -> QT6_MISO
- J1 pad 5: QT3_TX -> QT7_MOSI
- J4 pad 1: D3_SDA -> QT1_DAC
- R3 pad 2: Net-(SW2-A) -> Net-(SW2-C)
- SW1 pad 1: Net-(D7-A) -> unconnected-(SW1-A-Pad1)
- SW1 pad 3: unconnected-(SW1-C-Pad3) -> Net-(D7-A)
- SW2 pad 1: Net-(SW2-A) -> unconnected-(SW2-A-Pad1)
- SW2 pad 3: unconnected-(SW2-C-Pad3) -> Net-(SW2-C)
Routing:
- net QT7_MOSI: track 0.00 -> 208.2 mm
- net QT6_MISO: track 0.00 -> 181.5 mm
- net PWR_GND: track 12.4 -> 178.3 mm
- net QT5_SCK: track 0.00 -> 161.3 mm
- net QT4_RX: track 0.00 -> 137.8 mm
- net QT1_DAC: track 0.00 -> 128.5 mm
- net QT2: track 0.00 -> 116.0 mm
- net QT3_TX: track 0.00 -> 84.2 mm
- net PWR_3V3: track 12.4 -> 73.5 mm
- net Net-(D7-A): track 0.00 -> 59.0 mm
- net Net-(D1-K): track 0.00 -> 55.2 mm
- net Net-(D3-A): track 0.00 -> 53.3 mm
- net D1: track 0.00 -> 53.3 mm
- net D2: track 0.00 -> 46.2 mm
- net D3_SDA: track 0.00 -> 37.1 mm
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- added copper zone on F.Cu, net (none)
Other:
- board outline added: 139 x 74 mm
- board text added: "QTouch controller"
- board text added: "XIAO SAMD21"
