File: content/post/week-8/qtouch-board/qtouch-board.kicad_sch (KiCad schematic)
At the start: 18 parts, among them J1 Conn_PinSocket_1x05_P2.54mm_V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, J2 Conn_PinSocket_1x02_P2.54mm_V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, J3 Conn_PinSocket_1x03_P2.54mm_V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, J4 Conn_PinSocket_1x02_P2.54mm_V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, SW1 Switch_Slide_Top_CnK, SW2 Switch_Slide_Top_CnK, U1 SeeeduinoXIAO

Commit message: Catching up with documentation for weeks 7 and 8
Parts:
- removed J4: Conn_PinSocket_1x02_P2.54mm_Vertical_SMD, fab:PinSocket_1x02_P2.54mm_Vertical_SMD, symbol fab:Conn_PinSocket_1x02_P2.54mm_Vertical_SMD
- added H1, H2, H3: MountingHole_M3, fab:MountingHole_M3, symbol fab:MountingHole_M3
- added J10, J11, J4, J6, J7, J8, J9: Conn_PinHeader_1x01_P2.54mm_Vertical_THT_D1mm, fab:PinHeader_1x01_P2.54mm_Vertical_THT_D1mm, symbol fab:Conn_PinHeader_1x01_P2.54mm_Vertical_THT_D1mm
- added J5: Conn_Header_JST_PH_1x04_P2mm_Vertical_SMD, fab:Header_JST_PH_1x04_P2mm_Vertical_SMD, symbol fab:Conn_Header_JST_PH_1x04_P2mm_Vertical_SMD
- R1, R2, R3: value R_1206 -> R_1206_40
- R4: value R_1206 -> R_1206_80
Connections:
- net D3_SDA: now also J5.3
- net D4_SCL: now also J5.4
- net PWR_3V3: now also J5.2
- net PWR_GND: now also J5.1
- net QT1_DAC: now also J4.1 (Pin_1)
- net QT2: now also J6.1 (Pin_1)
- net QT3_TX: now also J7.1 (Pin_1)
- net QT4_RX: now also J8.1 (Pin_1)
- net QT5_SCK: now also J9.1 (Pin_1)
- net QT6_MISO: now also J10.1 (Pin_1)
- net QT7_MOSI: now also J11.1 (Pin_1)
- net at SW2.1 (A): no longer R3.2
- net at SW2.3 (C): now also R3.2
- net at SW1.1 (A): no longer D7.2 (A)
- net at SW1.3 (C): now also D7.2 (A)
Other:
- moved on the sheet: J1, J2, SW1, SW2
